File: Hardware/GPS_Shield.sch (EAGLE design)
At the start: 52 parts, among them J1 ARDUINO_R3_SHIELD, J2 USD_CONNECTOR, J3 GP-735-VERTICAL, U1 3.3V, U2 GP3906-TLP, U3 TXB0108

Commit message: Adding measures, cleaning up schematic
Parts:
- U1: value 3.3V -> APK2112-3.3V
Other:
- note added: "GP3906 VCC Range: 3.3V +/-5%"
- note added: "Input supplied by Arduino 5V"
- note removed: "5Vin Supplied by Arduino"
- moved on the sheet: C2

Commit message: Changing GP-735 module's VCC to 3.3V
Connections:
- net 3.3V: now also J3.VCC
- net 5V: no longer J3.VCC
Other:
- note added: "GP-735 VCC Range: 3.1V-5.5V"
Changed lines of the file:
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@@
 <part name="U3" library="SparkFun-DigitalIC" deviceset="TXB0108" device=""/>
 <part name="J3" library="SparkFun-RF" deviceset="GP-735" device="-VERTICAL"/>
-<part name="SUPPLY7" library="SparkFun-Aesthetics" deviceset="5V" device=""/>
 <part name="SUPPLY8" library="SparkFun-Aesthetics" deviceset="V_BATT" device=""/>
 <part name="SUPPLY6" library="SparkFun-Aesthetics" deviceset="V_BATT" device=""/>
@@
 <part name="P+6" library="SparkFun" deviceset="3.3V" device=""/>
 <part name="P+7" library="SparkFun" deviceset="3.3V" device=""/>
+<part name="P+11" library="SparkFun" deviceset="3.3V" device=""/>
 </parts>
 <sheets>
@@
 <text x="106.68" y="175.26" size="1.27" layer="97">GP3906 VCC
 Range: 3.3V +/-5%</text>
+<text x="137.16" y="175.26" size="1.27" layer="97">GP-735 VCC
+Range: 3.1V-5.5V</text>
 </plain>
 <instances>
@@
 <instance part="U3" gate="G$1" x="203.2" y="111.76" rot="MR0"/>
 <instance part="J3" gate="G$1" x="149.86" y="160.02"/>
-<instance part="SUPPLY7" gate="G$1" x="137.16" y="167.64"/>
 <instance part="SUPPLY8" gate="G$1" x="203.2" y="170.18" smashed="yes">
 <attribute name="VALUE" x="203.2" y="173.736" size="1.778" layer="96" align="bottom-center"/>
@@
 <instance part="P+6" gate="G$1" x="134.62" y="134.62"/>
 <instance part="P+7" gate="G$1" x="142.24" y="134.62"/>
+<instance part="P+11" gate="G$1" x="137.16" y="167.64"/>
 </instances>
 <busses>
@@
 <wire x1="142.24" y1="134.62" x2="142.24" y2="132.08" width="0.1524" layer="91"/>
 </segment>
+<segment>
+<pinref part="J3" gate="G$1" pin="VCC"/>
+<pinref part="P+11" gate="G$1" pin="3.3V"/>
+<wire x1="139.7" y1="165.1" x2="137.16" y2="165.1" width="0.1524" layer="91"/>
+<wire x1="137.16" y1="165.1" x2="137.16" y2="167.64" width="0.1524" layer="91"/>
+</segment>
 </net>
 <net name="5V" class="0">
 <segment>
-<pinref part="J3" gate="G$1" pin="VCC"/>
-<wire x1="139.7" y1="165.1" x2="137.16" y2="165.1" width="0.1524" layer="91"/>
-<wire x1="137.16" y1="165.1" x2="137.16" y2="167.64" width="0.1524" layer="91"/>
-<pinref part="SUPPLY7" gate="G$1" pin="5V"/>
-</segment>
-<segment>
 <pinref part="SJ3" gate="G$1" pin="3"/>

Commit message: Moving GP-735 connector to bottom side, marking DNP
Parts:
- J3: value GP-735-VERTICAL -> DNP (GP-735-VERTICAL)
Connections:
- net GPS_RST: now also JP18.5; no longer JP18.3
- net GPS_RX: now also JP18.4; no longer JP18.5
- net GPS_TX: now also JP18.3; no longer JP18.4
Changed lines of the file:
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@@
 <part name="JP5" library="SparkFun-Connectors" deviceset="M06" device="NO_SILK_FEMALE_PTH"/>
 <part name="U3" library="SparkFun-DigitalIC" deviceset="TXB0108" device=""/>
-<part name="J3" library="SparkFun-RF" deviceset="GP-735" device="-VERTICAL"/>
+<part name="J3" library="SparkFun-RF" deviceset="GP-735" device="-VERTICAL" value="DNP (GP-735-VERTICAL)"/>
 <part name="SUPPLY8" library="SparkFun-Aesthetics" deviceset="V_BATT" device=""/>
 <part name="SUPPLY6" library="SparkFun-Aesthetics" deviceset="V_BATT" device=""/>
@@
 </segment>
 <segment>
+<pinref part="JP18" gate="G$1" pin="4"/>
+<wire x1="180.34" y1="160.02" x2="177.8" y2="160.02" width="0.1524" layer="91"/>
+<label x="177.8" y="160.02" size="1.27" layer="95" rot="MR0" xref="yes"/>
+</segment>
+</net>
+<net name="GPS_TX" class="0">
+<segment>
+<pinref part="J3" gate="G$1" pin="TX"/>
+<wire x1="139.7" y1="162.56" x2="137.16" y2="162.56" width="0.1524" layer="91"/>
+<label x="137.16" y="162.56" size="1.27" layer="95" rot="R180" xref="yes"/>
+</segment>
+<segment>
+<pinref part="U3" gate="G$1" pin="A8"/>
+<wire x1="215.9" y1="99.06" x2="220.98" y2="99.06" width="0.1524" layer="91"/>
+<label x="220.98" y="99.06" size="1.27" layer="95" xref="yes"/>
+</segment>
+<segment>
+<pinref part="U2" gate="G$1" pin="TX"/>
+<wire x1="99.06" y1="162.56" x2="96.52" y2="162.56" width="0.1524" layer="91"/>
+<label x="96.52" y="162.56" size="1.27" layer="95" rot="R180" xref="yes"/>
+</segment>
+<segment>
+<pinref part="JP18" gate="G$1" pin="3"/>
+<wire x1="180.34" y1="162.56" x2="177.8" y2="162.56" width="0.1524" layer="91"/>
+<label x="177.8" y="162.56" size="1.27" layer="95" rot="MR0" xref="yes"/>
+</segment>
+</net>
+<net name="GPS_FIX" class="0">
+<segment>
+<pinref part="U2" gate="G$1" pin="3D_FIX"/>
+<wire x1="99.06" y1="157.48" x2="96.52" y2="157.48" width="0.1524" layer="91"/>
+<label x="96.52" y="157.48" size="1.27" layer="95" rot="R180" xref="yes"/>
+</segment>
+<segment>
+<pinref part="JP18" gate="G$1" pin="2"/>
+<wire x1="180.34" y1="165.1" x2="177.8" y2="165.1" width="0.1524" layer="91"/>
+<label x="177.8" y="165.1" size="1.27" layer="95" rot="MR0" xref="yes"/>
+</segment>
+<segment>
+<pinref part="SJ9" gate="G$1" pin="2"/>
+<wire x1="228.6" y1="175.26" x2="226.06" y2="175.26" width="0.1524" layer="91"/>
+<label x="226.06" y="175.26" size="1.27" layer="95" rot="R180" xref="yes"/>
+</segment>
+</net>
+<net name="GPS_RST" class="0">
+<segment>
+<pinref part="U2" gate="G$1" pin="RESET"/>
+<wire x1="99.06" y1="165.1" x2="96.52" y2="165.1" width="0.1524" layer="91"/>
+<label x="96.52" y="165.1" size="1.27" layer="95" rot="R180" xref="yes"/>
+</segment>
+<segment>
+<pinref part="J3" gate="G$1" pin="PWR_CTRL"/>
+<wire x1="139.7" y1="154.94" x2="137.16" y2="154.94" width="0.1524" layer="91"/>
+<label x="137.16" y="154.94" size="1.27" layer="95" rot="R180" xref="yes"/>
+</segment>
+<segment>
 <pinref part="JP18" gate="G$1" pin="5"/>
 <wire x1="180.34" y1="157.48" x2="177.8" y2="157.48" width="0.1524" layer="91"/>
@@
 </segment>
 </net>
-<net name="GPS_TX" class="0">
-<segment>
-<pinref part="J3" gate="G$1" pin="TX"/>
-<wire x1="139.7" y1="162.56" x2="137.16" y2="162.56" width="0.1524" layer="91"/>
-<label x="137.16" y="162.56" size="1.27" layer="95" rot="R180" xref="yes"/>
-</segment>
-<segment>
-<pinref part="U3" gate="G$1" pin="A8"/>
-<wire x1="215.9" y1="99.06" x2="220.98" y2="99.06" width="0.1524" layer="91"/>
-<label x="220.98" y="99.06" size="1.27" layer="95" xref="yes"/>
-</segment>
-<segment>
-<pinref part="U2" gate="G$1" pin="TX"/>
-<wire x1="99.06" y1="162.56" x2="96.52" y2="162.56" width="0.1524" layer="91"/>
-<label x="96.52" y="162.56" size="1.27" layer="95" rot="R180" xref="yes"/>
-</segment>
-<segment>
-<pinref part="JP18" gate="G$1" pin="4"/>
-<wire x1="180.34" y1="160.02" x2="177.8" y2="160.02" width="0.1524" layer="91"/>
-<label x="177.8" y="160.02" size="1.27" layer="95" rot="MR0" xref="yes"/>
-</segment>
-</net>
-<net name="GPS_FIX" class="0">
-<segment>
-<pinref part="U2" gate="G$1" pin="3D_FIX"/>
-<wire x1="99.06" y1="157.48" x2="96.52" y2="157.48" width="0.1524" layer="91"/>
-<label x="96.52" y="157.48" size="1.27" layer="95" rot="R180" xref="yes"/>
-</segment>
-<segment>
-<pinref part="JP18" gate="G$1" pin="2"/>
-<wire x1="180.34" y1="165.1" x2="177.8" y2="165.1" width="0.1524" layer="91"/>
-<label x="177.8" y="165.1" size="1.27" layer="95" rot="MR0" xref="yes"/>
-</segment>
-<segment>
-<pinref part="SJ9" gate="G$1" pin="2"/>
-<wire x1="228.6" y1="175.26" x2="226.06" y2="175.26" width="0.1524" layer="91"/>
-<label x="226.06" y="175.26" size="1.27" layer="95" rot="R180" xref="yes"/>
-</segment>
-</net>
-<net name="GPS_RST" class="0">
-<segment>
-<pinref part="U2" gate="G$1" pin="RESET"/>
-<wire x1="99.06" y1="165.1" x2="96.52" y2="165.1" width="0.1524" layer="91"/>
-<label x="96.52" y="165.1" size="1.27" layer="95" rot="R180" xref="yes"/>
-</segment>
-<segment>
-<pinref part="J3" gate="G$1" pin="PWR_CTRL"/>
-<wire x1="139.7" y1="154.94" x2="137.16" y2="154.94" width="0.1524" layer="91"/>
-<label x="137.16" y="154.94" size="1.27" layer="95" rot="R180" xref="yes"/>
-</segment>
-<segment>
-<pinref part="JP18" gate="G$1" pin="3"/>
-<wire x1="180.34" y1="162.56" x2="177.8" y2="162.56" width="0.1524" layer="91"/>
-<label x="177.8" y="162.56" size="1.27" layer="95" rot="MR0" xref="yes"/>
-</segment>
-</net>
